Commit message: fix urdf for simulation purposes
Added fake effort limits
Changed Gazebo Classic plugin to Gazebo Fortress

File: ar_description/urdf/ar_gazebo.urdf.xacro (robot description, xacro)
@@ -16,5 +16,5 @@
   <xacro:ar_ros2_control
     ar_model="$(arg ar_model)"
-    plugin_name="gazebo_ros2_control/GazeboSystem"
+    plugin_name="ign_ros2_control/IgnitionSystem"
     serial_port="None"
     calibrate="False"
@@ -24,10 +24,10 @@
   <xacro:ar_gripper_ros2_control
     name="ARGripperGazeboSystem"
-    plugin_name="gazebo_ros2_control/GazeboSystem"
+    plugin_name="ign_ros2_control/IgnitionSystem"
     serial_port="None"
   />
   <gazebo reference="world" />
   <gazebo>
-    <plugin filename="libgazebo_ros2_control.so" name="gazebo_ros2_control">
+    <plugin filename="libign_ros2_control-system.so" name="ign_ros2_control::IgnitionROS2ControlPlugin">
       <parameters>$(arg simulation_controllers)</parameters>
     </plugin>

File: ar_description/urdf/ar_gripper_macro.xacro (robot description, xacro)
@@ -72,5 +72,5 @@
       <child link="gripper_jaw1_link"/>
       <axis xyz="1 0 0"/>
-      <limit lower="-0.014" upper="0" effort="0" velocity="0.1"/>
+      <limit lower="-0.014" upper="0" effort="50" velocity="0.1"/>
     </joint>
     <joint name="gripper_jaw2_joint" type="prismatic">
@@ -79,5 +79,5 @@
       <child link="gripper_jaw2_link"/>
       <axis xyz="1 0 0"/>
-      <limit lower="-0.014" upper="0" effort="0" velocity="0.1"/>
+      <limit lower="-0.014" upper="0" effort="50" velocity="0.1"/>
       <mimic joint="gripper_jaw1_joint" multiplier="1" offset="0"/>
     </joint>

File: ar_description/urdf/ar_macro.xacro (robot description, xacro)
@@ -61,5 +61,5 @@
       <child link="link_1"/>
       <axis xyz="0 0 1"/>
-      <limit lower="${robot_parameters['j1_limit_min']}" upper="${robot_parameters['j1_limit_max']}" effort="0" velocity="0.5"/>
+      <limit lower="${robot_parameters['j1_limit_min']}" upper="${robot_parameters['j1_limit_max']}" effort="50" velocity="0.5"/>
     </joint>
     <link name="link_2">
@@ -90,5 +90,5 @@
       <child link="link_2"/>
       <axis xyz="0 0 -1"/>
-      <limit lower="${robot_parameters['j2_limit_min']}" upper="${robot_parameters['j2_limit_max']}" effort="0.5" velocity="0.5"/>
+      <limit lower="${robot_parameters['j2_limit_min']}" upper="${robot_parameters['j2_limit_max']}" effort="50" velocity="0.5"/>
     </joint>
     <link name="link_3">
@@ -119,5 +119,5 @@
       <child link="link_3"/>
       <axis xyz="0 0 -1"/>
-      <limit lower="${robot_parameters['j3_limit_min']}" upper="${robot_parameters['j3_limit_max']}" effort="0" velocity="0.5"/>
+      <limit lower="${robot_parameters['j3_limit_min']}" upper="${robot_parameters['j3_limit_max']}" effort="50" velocity="0.5"/>
     </joint>
     <link name="link_4">
@@ -148,5 +148,5 @@
       <child link="link_4"/>
       <axis xyz="0 0 -1"/>
-      <limit lower="${robot_parameters['j4_limit_min']}" upper="${robot_parameters['j4_limit_max']}" effort="0" velocity="0.5"/>
+      <limit lower="${robot_parameters['j4_limit_min']}" upper="${robot_parameters['j4_limit_max']}" effort="50" velocity="0.5"/>
     </joint>
     <link name="link_5">
@@ -177,5 +177,5 @@
       <child link="link_5"/>
       <axis xyz="1 0 0"/>
-      <limit lower="${robot_parameters['j5_limit_min']}" upper="${robot_parameters['j5_limit_max']}" effort="0" velocity="1.0"/>
+      <limit lower="${robot_parameters['j5_limit_min']}" upper="${robot_parameters['j5_limit_max']}" effort="50" velocity="1.0"/>
     </joint>
     <link name="link_6">
@@ -206,5 +206,5 @@
       <child link="link_6"/>
       <axis xyz="0 0 1"/>
-      <limit lower="${robot_parameters['j6_limit_min']}" upper="${robot_parameters['j6_limit_max']}" effort="0" velocity="1.0"/>
+      <limit lower="${robot_parameters['j6_limit_min']}" upper="${robot_parameters['j6_limit_max']}" effort="50" velocity="1.0"/>
     </joint>
     <!-- center of the end effector mounting surface on link_6 -->
