Commit message: refactor(robot): streamline AR4 configuration and simulation setup
- Reduced camera resolution and modified object positions in gazebo scene description.
- Moved `xacro_args.yaml` to `urdf` and `srdf` folders.
- Added gripper grasp point link and joint in URDF for enhanced grasping simulation.
- Switched from Gazebo to Ignition Gazebo in launch configurations.
- Updated `ar_moveit_config` to include `controllers.yaml` and adjusted controller references.
- Introduced `jspg.launch.py` for joint state publisher GUI integration.
- Relocated and renamed SRDF xacro arguments for better file organization.

File: ar_description/urdf/ar_gripper_macro.xacro (robot description, xacro)
@@ -67,4 +67,10 @@
       </inertial>
     </link>
+    <link name="gripper_grasp_point"/>
+    <joint name="gripper_grasp_point_joint" type="fixed">
+      <origin xyz="0.0 0.0 0.055" rpy="0.0 0.0 0.0" />
+      <child link="gripper_grasp_point"/>
+      <parent link="ee_link"/>
+    </joint>
     <joint name="gripper_jaw1_joint" type="prismatic">
       <origin xyz="0.0 -0.036 0" rpy="0.0 0.0 0.0"/>
